File: rev1/framework.kicad_pcb (KiCad board)
At the start: 2 copper layers, 238.1 x 375.5 mm, 197 parts, among them J1 AVR-ISP-6, J2 USB_C_Receptacle_USB2.0, SW1 SW_Push, SW10 SW_Push_45deg, SW11 SW_Push_45deg, SW12 SW_Push_45deg, SW13 SW_Push_45deg, SW14 SW_Push_45deg, SW15 SW_Push_45deg, SW16 SW_Push_45deg, SW17 SW_Push_45deg, SW18 SW_Push_45deg, SW19 SW_Push_45deg, SW2 SW_Push, SW20 SW_Push_45deg, SW21 SW_Push_45deg, SW22 SW_Push_45deg, SW23 SW_Push_45deg, SW24 SW_Push_45deg, SW25 SW_Push_45deg, SW26 SW_Push_45deg, SW27 SW_Push_45deg, SW28 SW_Push_45deg, SW29 SW_Push_45deg, SW3 SW_Push_45deg, SW30 SW_Push_45deg, SW31 SW_Push_45deg, SW32 SW_Push_45deg, SW33 SW_Push_45deg, SW34 SW_Push_45deg, SW35 SW_Push_45deg, SW36 SW_Push_45deg, SW37 SW_Push_45deg, SW38 SW_Push_45deg, SW39 SW_Push_45deg, SW4 SW_Push_45deg, SW40 SW_Push_45deg, SW41 SW_Push_45deg, SW42 SW_Push_45deg, SW43 SW_Push_45deg, SW44 SW_Push_45deg, SW45 SW_Push_45deg, SW46 SW_Push_45deg, SW47 SW_Push_45deg, SW48 SW_Push_45deg, SW49 SW_Push_45deg, SW5 SW_Push_45deg, SW50 SW_Push_45deg, SW51 SW_Push_45deg, SW52 SW_Push_45deg, SW53 SW_Push_45deg, SW54 SW_Push_45deg, SW55 SW_Push_45deg, SW56 SW_Push_45deg, SW57 SW_Push_45deg, SW58 SW_Push_45deg, SW59 SW_Push_45deg, SW6 SW_Push_45deg, SW60 SW_Push_45deg, SW61 SW_Push_45deg, SW62 SW_Push_45deg, SW63 Rotary_Encoder_Switch, SW64 SW_Push_45deg, SW65 SW_Push_45deg, SW7 SW_Push_45deg, SW8 SW_Push_45deg, SW9 SW_Push_45deg, U1 ATmega328P-PU, Y1 16M

Commit message: reformatted to 48 key iso-ish thing
Parts:
- removed D38, D42, D44, D46, D48, D50, D52, D54, D56, D58, D60, D62: D, framework:D_DO-35_SOD27_P7.62mm_Horizontal
- removed the REF** at (333.0, 363.1)
- removed the REF** at (217.6, 361.9)
- removed the REF** at (314.0, 234.9)
- removed the REF** at (102.1, 363.1)
- removed the REF** at (333.0, 118.6)
- removed the REF** at (236.6, 321.8)
- removed the REF** at (198.5, 321.8)
- removed the REF** at (217.6, 226.6)
- removed the REF** at (217.6, 321.8)
- removed the REF** at (333.0, 227.8)
- removed the REF** at (102.1, 227.8)
- removed the REF** at (314.0, 370.3)
- removed SW38, SW42, SW44, SW46, SW48, SW50, SW52, SW55, SW57, SW59, SW61, SW62, SW64, SW65: SW_Push_45deg, framework:Kailh_socket_MX_no_fsilk
- removed SW63: Rotary_Encoder_Switch, framework:RotaryEncoder_Alps_EC11E-Switch_Vertical_H20mm
- removed the mouse-bite-2mm-slot at (317.6, 201.8)
- removed the mouse-bite-2mm-slot at (317.6, 337.1)
- added REF**: MountingHole_2.2mm_M2, MountingHole:MountingHole_2.2mm_M2, F.Cu at (208.1, 210.4)
- added REF**: MountingHole_2.2mm_M2, MountingHole:MountingHole_2.2mm_M2, F.Cu at (283.3, 341.6)
- added REF**: MountingHole_2.2mm_M2, MountingHole:MountingHole_2.2mm_M2, F.Cu at (283.3, 205.9)
- added REF**: MountingHole_2.2mm_M2, MountingHole:MountingHole_2.2mm_M2, F.Cu at (208.1, 345.8)
- added REF**: MountingHole_2.2mm_M2, MountingHole:MountingHole_2.2mm_M2, F.Cu at (95.1, 211.6)
- added REF**: MountingHole_2.2mm_M2, MountingHole:MountingHole_2.2mm_M2, F.Cu at (95.1, 346.9)
- moved G*** 110.4 mm to (109.5, 337.1)
- moved REF** 52.3 mm to (283.3, 373.1)
- moved REF** 52.3 mm to (283.3, 325.5)
- moved REF** 52.3 mm to (283.3, 181.0)
- moved REF** 52.3 mm to (283.3, 451.7)
- moved REF** 52.3 mm to (283.3, 190.2)
- moved REF** 52.3 mm to (283.3, 237.8)
- moved REF** 52.3 mm to (283.3, 316.4)
- moved SW2 48.0 mm to (278.7, 200.8), turned to -90 degrees
- moved SW1 42.2 mm to (278.7, 190.6), turned to -90 degrees
- moved G*** 41.3 mm to (275.7, 214.2)
- moved REF** 34.7 mm to (283.3, 83.4)
- moved G*** 28.2 mm to (258.6, 315.9)
- moved G*** 28.2 mm to (261.9, 311.2)
- moved G*** 28.2 mm to (233.9, 312.7)
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Connections:
- C4 pad 1: Net-(C4-Pad1) -> (no net)
- C5 pad 1: Net-(C5-Pad1) -> (no net)
- D1 pad 1: Net-(D1-Pad1) -> (no net)
- D10 pad 2: Net-(D10-Pad2) -> (no net)
- D11 pad 2: Net-(D11-Pad2) -> (no net)
- D12 pad 2: Net-(D12-Pad2) -> (no net)
- D13 pad 2: Net-(D13-Pad2) -> (no net)
- D14 pad 2: Net-(D14-Pad2) -> (no net)
- D15 pad 2: Net-(D15-Pad2) -> (no net)
- D16 pad 2: Net-(D16-Pad2) -> (no net)
- D17 pad 2: Net-(D17-Pad2) -> (no net)
- D18 pad 2: Net-(D18-Pad2) -> (no net)
- D19 pad 2: Net-(D19-Pad2) -> (no net)
- D2 pad 1: Net-(D2-Pad1) -> (no net)
- D20 pad 2: Net-(D20-Pad2) -> (no net)
- D21 pad 2: Net-(D21-Pad2) -> (no net)
- D22 pad 2: Net-(D22-Pad2) -> (no net)
- D23 pad 2: Net-(D23-Pad2) -> (no net)
- D24 pad 2: Net-(D24-Pad2) -> (no net)
- D25 pad 2: Net-(D25-Pad2) -> (no net)
- D26 pad 2: Net-(D26-Pad2) -> (no net)
- D27 pad 2: Net-(D27-Pad2) -> (no net)
- D28 pad 2: Net-(D28-Pad2) -> (no net)
- D29 pad 2: Net-(D29-Pad2) -> (no net)
- D3 pad 2: Net-(D3-Pad2) -> (no net)
- D30 pad 2: Net-(D30-Pad2) -> (no net)
- D31 pad 2: Net-(D31-Pad2) -> (no net)
- D32 pad 2: Net-(D32-Pad2) -> (no net)
- D33 pad 2: Net-(D33-Pad2) -> (no net)
- D34 pad 2: Net-(D34-Pad2) -> (no net)
- D35 pad 2: Net-(D35-Pad2) -> (no net)
- D36 pad 2: Net-(D36-Pad2) -> (no net)
- D37 pad 2: Net-(D37-Pad2) -> (no net)
- D39 pad 2: Net-(D39-Pad2) -> (no net)
- D4 pad 2: Net-(D4-Pad2) -> (no net)
- D40 pad 2: Net-(D40-Pad2) -> (no net)
- D41 pad 2: Net-(D41-Pad2) -> (no net)
- D43 pad 2: Net-(D43-Pad2) -> (no net)
- D45 pad 2: Net-(D45-Pad2) -> (no net)
- D47 pad 2: Net-(D47-Pad2) -> (no net)
- D49 pad 2: Net-(D49-Pad2) -> (no net)
- D5 pad 2: Net-(D5-Pad2) -> (no net)
- D51 pad 2: Net-(D51-Pad2) -> (no net)
- D53 pad 2: Net-(D53-Pad2) -> (no net)
- D55 pad 2: Net-(D55-Pad2) -> (no net)
- D57 pad 2: Net-(D57-Pad2) -> (no net)
- D59 pad 2: Net-(D59-Pad2) -> (no net)
- D6 pad 2: Net-(D6-Pad2) -> (no net)
- D61 pad 2: Net-(D61-Pad2) -> (no net)
- D7 pad 2: Net-(D7-Pad2) -> (no net)
- D8 pad 2: Net-(D8-Pad2) -> (no net)
- D9 pad 2: Net-(D9-Pad2) -> (no net)
- J2 pad A5: Net-(J2-PadA5) -> (no net)
- J2 pad A6: Net-(D1-Pad1) -> Net-(D1-K)
- J2 pad A7: Net-(D2-Pad1) -> Net-(D2-K)
- J2 pad A8: Net-(J2-PadA8) -> (no net)
- J2 pad B5: Net-(J2-PadB5) -> (no net)
- J2 pad B6: Net-(D1-Pad1) -> Net-(D1-K)
- J2 pad B7: Net-(D2-Pad1) -> Net-(D2-K)
- J2 pad B8: Net-(J2-PadB8) -> (no net)
- R2 pad 2: Net-(D2-Pad1) -> Net-(D2-K)
- R3 pad 2: Net-(D1-Pad1) -> Net-(D1-K)
- R5 pad 2: Net-(J2-PadB5) -> Net-(J2-CC2)
- R6 pad 2: Net-(J2-PadA5) -> Net-(J2-CC1)
- SW10 pad 1: Net-(D10-Pad2) -> Net-(D10-A)
- SW11 pad 1: Net-(D11-Pad2) -> Net-(D11-A)
- SW12 pad 1: Net-(D12-Pad2) -> Net-(D12-A)
- SW13 pad 1: Net-(D13-Pad2) -> Net-(D13-A)
- SW14 pad 1: Net-(D14-Pad2) -> Net-(D14-A)
- SW15 pad 1: Net-(D15-Pad2) -> Net-(D15-A)
- SW16 pad 1: Net-(D16-Pad2) -> Net-(D16-A)
- SW17 pad 1: Net-(D17-Pad2) -> Net-(D17-A)
- SW18 pad 1: Net-(D18-Pad2) -> Net-(D18-A)
- SW19 pad 1: Net-(D19-Pad2) -> Net-(D19-A)
- SW20 pad 1: Net-(D20-Pad2) -> Net-(D20-A)
- SW21 pad 1: Net-(D21-Pad2) -> Net-(D21-A)
- SW22 pad 1: Net-(D22-Pad2) -> Net-(D22-A)
- SW23 pad 1: Net-(D23-Pad2) -> Net-(D23-A)
- SW24 pad 1: Net-(D24-Pad2) -> Net-(D24-A)
- SW25 pad 1: Net-(D25-Pad2) -> Net-(D25-A)
- SW26 pad 1: Net-(D26-Pad2) -> Net-(D26-A)
- SW27 pad 1: Net-(D27-Pad2) -> Net-(D27-A)
- SW28 pad 1: Net-(D28-Pad2) -> Net-(D28-A)
- SW29 pad 1: Net-(D29-Pad2) -> Net-(D29-A)
- SW3 pad 1: Net-(D3-Pad2) -> Net-(D3-A)
- SW30 pad 1: Net-(D30-Pad2) -> Net-(D30-A)
- SW31 pad 1: Net-(D31-Pad2) -> Net-(D31-A)
- SW32 pad 1: Net-(D32-Pad2) -> Net-(D32-A)
- SW33 pad 1: Net-(D33-Pad2) -> Net-(D33-A)
- SW34 pad 1: Net-(D34-Pad2) -> Net-(D34-A)
- SW35 pad 1: Net-(D35-Pad2) -> Net-(D35-A)
- SW36 pad 1: Net-(D36-Pad2) -> Net-(D36-A)
- SW37 pad 1: Net-(D37-Pad2) -> Net-(D37-A)
- SW39 pad 1: Net-(D39-Pad2) -> Net-(D39-A)
- SW4 pad 1: Net-(D4-Pad2) -> Net-(D4-A)
- SW40 pad 1: Net-(D40-Pad2) -> Net-(D40-A)
- SW41 pad 1: Net-(D41-Pad2) -> Net-(D41-A)
- SW43 pad 1: Net-(D43-Pad2) -> Net-(D43-A)
- SW45 pad 1: Net-(D45-Pad2) -> Net-(D45-A)
- SW47 pad 1: Net-(D47-Pad2) -> Net-(D47-A)
- SW49 pad 1: Net-(D49-Pad2) -> Net-(D49-A)
- SW5 pad 1: Net-(D5-Pad2) -> Net-(D5-A)
- SW51 pad 1: Net-(D51-Pad2) -> Net-(D51-A)
- SW53 pad 1: Net-(D53-Pad2) -> Net-(D53-A)
- SW54 pad 1: Net-(D55-Pad2) -> Net-(D55-A)
- SW56 pad 1: Net-(D57-Pad2) -> Net-(D57-A)
- SW58 pad 1: Net-(D59-Pad2) -> Net-(D59-A)
- SW6 pad 1: Net-(D6-Pad2) -> Net-(D6-A)
- SW60 pad 1: Net-(D61-Pad2) -> Net-(D61-A)
- SW7 pad 1: Net-(D7-Pad2) -> Net-(D7-A)
- SW8 pad 1: Net-(D8-Pad2) -> Net-(D8-A)
- SW9 pad 1: Net-(D9-Pad2) -> Net-(D9-A)
- U1 pad 10: Net-(C4-Pad1) -> Net-(U1-XTAL2/PB7)
- U1 pad 21: Net-(U1-Pad21) -> (no net)
- U1 pad 9: Net-(C5-Pad1) -> Net-(U1-XTAL1/PB6)
- Y1 pad 1: Net-(C4-Pad1) -> Net-(U1-XTAL2/PB7)
- Y1 pad 2: Net-(C5-Pad1) -> Net-(U1-XTAL1/PB6)
Routing:
- net c5: track 404.6 -> 148.7 mm, vias 4 -> 3
- net c4: track 344.2 -> 163.8 mm, vias 4 -> 2
- net Net-(D61-Pad2): track 161.3 -> 0.00 mm
- net Net-(D52-Pad2): track 160.8 -> 0.00 mm
- net Net-(D32-A): track 0.00 -> 146.4 mm
- net Net-(D62-Pad2): track 144.1 -> 0.00 mm
- net Net-(D50-Pad2): track 143.5 -> 0.00 mm
- net Net-(D51-A): track 0.00 -> 141.5 mm
- net Net-(D61-A): track 0.00 -> 140.0 mm
- net Net-(D51-Pad2): track 132.9 -> 0.00 mm
- net Net-(D12-A): track 0.00 -> 132.4 mm
- net Net-(D31-A): track 0.00 -> 129.9 mm
- net Net-(D32-Pad2): track 129.0 -> 0.00 mm
- net Net-(D12-Pad2): track 127.9 -> 0.00 mm
- net Net-(D11-A): track 0.00 -> 126.8 mm
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- removed copper zone on B.Cu, net (none)
- removed copper zone on F.Cu, net (none)
Other:
- board size 238.1 x 375.5 mm -> 195.3 x 375.5 mm
- net class Default removed
- rule pad_to_mask_clearance: 0.051 -> 0
- board text added: "cool awesome baller, sooooo so cool and awesome. the best."
- board text added: "newk board"
